File: proxima.sch (KiCad schematic (older format))
At the start: 6 parts

Commit message: switching
Parts:
- added J?: Conn_01x03_Female, symbol Connector:Conn_01x03_Female
- added K?: DIPxx-1Axx-12x, Relay_THT:Relay_StandexMeder_DIP_LowProfile, symbol Relay:DIPxx-1Axx-12x
- added Q?: BC547, Package_TO_SOT_THT:TO-92_Inline, symbol Transistor_BJT:BC547
- added R?: 1k, symbol Device:R_US
Connections:
- net labels added: GND
- wire segments 16 -> 25
Other:
- moved on the sheet: C?, D?, R?
Changed lines of the file:
@@
 L Device:C C?
 U 1 1 6362C072
-P 1150 2700
-F 0 "C?" V 898 2700 50  0000 C CNN
-F 1 "C" V 989 2700 50  0000 C CNN
-F 2 "" H 1188 2550 50  0001 C CNN
-F 3 "~" H 1150 2700 50  0001 C CNN
-	1    1150 2700
+P 4900 3050
+F 0 "C?" V 4648 3050 50  0000 C CNN
+F 1 "C" V 4739 3050 50  0000 C CNN
+F 2 "" H 4938 2900 50  0001 C CNN
+F 3 "~" H 4900 3050 50  0001 C CNN
+	1    4900 3050
 	0    1    1    0
 $EndComp
@@
 L Device:CP1 C?
 U 1 1 6362C51F
-P 3150 3250
-F 0 "C?" H 3265 3296 50  0000 L CNN
-F 1 "470" H 3265 3205 50  0000 L CNN
-F 2 "" H 3150 3250 50  0001 C CNN
-F 3 "~" H 3150 3250 50  0001 C CNN
-	1    3150 3250
+P 6900 3600
+F 0 "C?" H 7015 3646 50  0000 L CNN
+F 1 "470" H 7015 3555 50  0000 L CNN
+F 2 "" H 6900 3600 50  0001 C CNN
+F 3 "~" H 6900 3600 50  0001 C CNN
+	1    6900 3600
 	1    0    0    -1
 $EndComp
@@
 L Device:D_Bridge_+-AA D?
 U 1 1 6362D2C4
-P 1850 2850
-F 0 "D?" H 2194 2896 50  0000 L CNN
-F 1 "D_Bridge_+-AA" H 2194 2805 50  0000 L CNN
-F 2 "" H 1850 2850 50  0001 C CNN
-F 3 "~" H 1850 2850 50  0001 C CNN
-	1    1850 2850
+P 5600 3200
+F 0 "D?" H 5944 3246 50  0000 L CNN
+F 1 "D_Bridge_+-AA" H 5944 3155 50  0000 L CNN
+F 2 "" H 5600 3200 50  0001 C CNN
+F 3 "~" H 5600 3200 50  0001 C CNN
+	1    5600 3200
 	1    0    0    -1
 $EndComp
@@
 L Diode:DZ2S051X0L D?
 U 1 1 6362E947
-P 2700 3250
-F 0 "D?" V 2654 3329 50  0000 L CNN
-F 1 "DZ2S051X0L" V 2745 3329 50  0000 L CNN
-F 2 "Diode_SMD:D_SOD-523" H 2700 3075 50  0001 C CNN
-F 3 "https://industrial.panasonic.com/content/data/SC/ds/ds4/DZ2S05100L_E.pdf" H 2700 3250 50  0001 C CNN
-	1    2700 3250
+P 6450 3600
+F 0 "D?" V 6404 3679 50  0000 L CNN
+F 1 "DZ2S051X0L" V 6495 3679 50  0000 L CNN
+F 2 "Diode_SMD:D_SOD-523" H 6450 3425 50  0001 C CNN
+F 3 "https://industrial.panasonic.com/content/data/SC/ds/ds4/DZ2S05100L_E.pdf" H 6450 3600 50  0001 C CNN
+	1    6450 3600
 	0    1    1    0
 $EndComp
@@
 L Device:R_US R?
 U 1 1 6362F5CB
-P 1150 3000
-F 0 "R?" V 945 3000 50  0000 C CNN
-F 1 "470K" V 1036 3000 50  0000 C CNN
-F 2 "" V 1190 2990 50  0001 C CNN
-F 3 "~" H 1150 3000 50  0001 C CNN
-	1    1150 3000
+P 4900 3350
+F 0 "R?" V 4695 3350 50  0000 C CNN
+F 1 "470K" V 4786 3350 50  0000 C CNN
+F 2 "" V 4940 3340 50  0001 C CNN
+F 3 "~" H 4900 3350 50  0001 C CNN
+	1    4900 3350
 	0    1    1    0
 $EndComp
@@
 L Device:R_US R?
 U 1 1 63630132
-P 1150 3400
-F 0 "R?" V 945 3400 50  0000 C CNN
-F 1 "100" V 1036 3400 50  0000 C CNN
-F 2 "" V 1190 3390 50  0001 C CNN
-F 3 "~" H 1150 3400 50  0001 C CNN
-	1    1150 3400
+P 4900 3750
+F 0 "R?" V 4695 3750 50  0000 C CNN
+F 1 "100" V 4786 3750 50  0000 C CNN
+F 2 "" V 4940 3740 50  0001 C CNN
+F 3 "~" H 4900 3750 50  0001 C CNN
+	1    4900 3750
 	0    1    1    0
 $EndComp
@@
 L power:AC #PWR?
 U 1 1 6363069B
-P 650 2700
-F 0 "#PWR?" H 650 2600 50  0001 C CNN
-F 1 "AC" H 650 2975 50  0000 C CNN
-F 2 "" H 650 2700 50  0001 C CNN
-F 3 "" H 650 2700 50  0001 C CNN
-	1    650  2700
-	1    0    0    -1
-$EndComp
-Wire Wire Line
-	1300 3000 1300 2850
-Wire Wire Line
-	1850 2550 1450 2550
-Wire Wire Line
-	1450 2550 1450 2850
-Wire Wire Line
-	1450 2850 1300 2850
-Connection ~ 1300 2850
-Wire Wire Line
-	1300 2850 1300 2700
-Wire Wire Line
-	1000 3000 1000 2700
-Wire Wire Line
-	650  2700 1000 2700
-Connection ~ 1000 2700
-Wire Wire Line
-	2150 2850 2700 2850
-Wire Wire Line
-	2700 2850 2700 3100
-Wire Wire Line
-	2700 3400 1550 3400
-Wire Wire Line
-	1550 3400 1550 2850
-Wire Wire Line
-	2700 3400 3150 3400
-Connection ~ 2700 3400
-Wire Wire Line
-	3150 3100 3150 2850
-Wire Wire Line
-	3150 2850 2700 2850
-Connection ~ 2700 2850
-Wire Wire Line
-	1550 3400 1300 3400
-Connection ~ 1550 3400
-Wire Wire Line
-	1000 3400 800  3400
+P 4400 3050
+F 0 "#PWR?" H 4400 2950 50  0001 C CNN
+F 1 "AC" H 4400 3325 50  0000 C CNN
+F 2 "" H 4400 3050 50  0001 C CNN
+F 3 "" H 4400 3050 50  0001 C CNN
+	1    4400 3050
+	1    0    0    -1
+$EndComp
+Wire Wire Line
+	5050 3350 5050 3200
+Wire Wire Line
+	5600 2900 5200 2900
+Wire Wire Line
+	5200 2900 5200 3200
+Wire Wire Line
+	5200 3200 5050 3200
+Connection ~ 5050 3200
+Wire Wire Line
+	5050 3200 5050 3050
+Wire Wire Line
+	4750 3350 4750 3050
+Wire Wire Line
+	4400 3050 4750 3050
+Connection ~ 4750 3050
+Wire Wire Line
+	5900 3200 6450 3200
+Wire Wire Line
+	6450 3200 6450 3450
+Wire Wire Line
+	6450 3750 5300 3750
+Wire Wire Line
+	5300 3750 5300 3200
+Wire Wire Line
+	6450 3750 6900 3750
+Connection ~ 6450 3750
+Wire Wire Line
+	6900 3450 6900 3200
+Wire Wire Line
+	6900 3200 6450 3200
+Connection ~ 6450 3200
+Wire Wire Line
+	5300 3750 5050 3750
+Connection ~ 5300 3750
+Wire Wire Line
+	4750 3750 4550 3750
+$Comp
+L Relay:DIPxx-1Axx-12x K?
+U 1 1 63693C13
+P 8350 3400
+F 0 "K?" H 8680 3446 50  0000 L CNN
+F 1 "DIPxx-1Axx-12x" H 8680 3355 50  0000 L CNN
+F 2 "Relay_THT:Relay_StandexMeder_DIP_LowProfile" H 8700 3350 50  0001 L CNN
+F 3 "https://standexelectronics.com/wp-content/uploads/datasheet_reed_relay_DIP.pdf" H 8350 3400 50  0001 C CNN
+	1    8350 3400
+	1    0    0    -1
+$EndComp
+Wire Wire Line
+	8150 3100 7750 3100
+Wire Wire Line
+	6900 3100 6900 3200
+Connection ~ 6900 3200
+$Comp
+L Transistor_BJT:BC547 Q?
+U 1 1 63695DED
+P 7950 4300
+F 0 "Q?" H 8141 4346 50  0000 L CNN
+F 1 "BC547" H 8141 4255 50  0000 L CNN
+F 2 "Package_TO_SOT_THT:TO-92_Inline" H 8150 4225 50  0001 L CIN
+F 3 "http://www.fairchildsemi.com/ds/BC/BC547.pdf" H 7950 4300 50  0001 L CNN
+	1    7950 4300
+	1    0    0    -1
+$EndComp
+$Comp
+L Connector:Conn_01x03_Female J?
+U 1 1 636A603E
+P 6500 4300
+F 0 "J?" H 6392 3975 50  0000 C CNN
+F 1 "Conn_01x03_Female" H 6392 4066 50  0000 C CNN
+F 2 "" H 6500 4300 50  0001 C CNN
+F 3 "~" H 6500 4300 50  0001 C CNN
+	1    6500 4300
+	-1   0    0    1
+$EndComp
+$Comp
+L Device:R_US R?
+U 1 1 636ACF39
+P 7300 4300
+F 0 "R?" V 7095 4300 50  0000 C CNN
+F 1 "1k" V 7186 4300 50  0000 C CNN
+F 2 "" V 7340 4290 50  0001 C CNN
+F 3 "~" H 7300 4300 50  0001 C CNN
+	1    7300 4300
+	0    1    1    0
+$EndComp
+$Comp
+L power:GND #PWR?
+U 1 1 636B5108
+P 6900 3750
+F 0 "#PWR?" H 6900 3500 50  0001 C CNN
+F 1 "GND" H 6905 3577 50  0000 C CNN
+F 2 "" H 6900 3750 50  0001 C CNN
+F 3 "" H 6900 3750 50  0001 C CNN
+	1    6900 3750
+	1    0    0    -1
+$EndComp
+Connection ~ 6900 3750
+$Comp
+L power:GND #PWR?
+U 1 1 636B5B8D
+P 8050 4500
+F 0 "#PWR?" H 8050 4250 50  0001 C CNN
+F 1 "GND" H 8055 4327 50  0000 C CNN
+F 2 "" H 8050 4500 50  0001 C CNN
+F 3 "" H 8050 4500 50  0001 C CNN
+	1    8050 4500
+	1    0    0    -1
+$EndComp
+Wire Wire Line
+	7450 4300 7750 4300
+Wire Wire Line
+	6700 4300 7150 4300
+Wire Wire Line
+	8050 4100 8050 3700
+Wire Wire Line
+	8050 3700 8150 3700
+$Comp
+L power:GND #PWR?
+U 1 1 636B6E73
+P 6700 4400
+F 0 "#PWR?" H 6700 4150 50  0001 C CNN
+F 1 "GND" H 6705 4227 50  0000 C CNN
+F 2 "" H 6700 4400 50  0001 C CNN
+F 3 "" H 6700 4400 50  0001 C CNN
+	1    6700 4400
+	1    0    0    -1
+$EndComp
+Wire Wire Line
+	7750 3100 7750 4200
+Wire Wire Line
+	7750 4200 6700 4200
+Connection ~ 7750 3100
+Wire Wire Line
+	7750 3100 6900 3100
 $EndSCHEMATC

Commit message: switching relay diode
Parts:
- added D?: 1N4007, Diode_THT:D_DO-41_SOD81_P10.16mm_Horizontal, symbol Diode:1N4007
Connections:
- wire segments 25 -> 29
Changed lines of the file:
@@
 $EndComp
 Wire Wire Line
-	8150 3100 7750 3100
+	8150 3100 7850 3100
 Wire Wire Line
 	6900 3100 6900 3200
@@
 	6700 4300 7150 4300
 Wire Wire Line
-	8050 4100 8050 3700
-Wire Wire Line
 	8050 3700 8150 3700
 $Comp
@@
 Wire Wire Line
 	7750 3100 6900 3100
+$Comp
+L Diode:1N4007 D?
+U 1 1 636B8955
+P 7850 3750
+F 0 "D?" V 7804 3829 50  0000 L CNN
+F 1 "1N4007" V 7895 3829 50  0000 L CNN
+F 2 "Diode_THT:D_DO-41_SOD81_P10.16mm_Horizontal" H 7850 3575 50  0001 C CNN
+F 3 "http://www.vishay.com/docs/88503/1n4001.pdf" H 7850 3750 50  0001 C CNN
+	1    7850 3750
+	0    1    1    0
+$EndComp
+Wire Wire Line
+	7850 3900 8050 3900
+Wire Wire Line
+	8050 3700 8050 3900
+Connection ~ 8050 3900
+Wire Wire Line
+	8050 3900 8050 4100
+Wire Wire Line
+	7850 3600 7850 3100
+Connection ~ 7850 3100
+Wire Wire Line
+	7850 3100 7750 3100
 $EndSCHEMATC
